Commit message: 20191017

File: turtlebot-kinetic/turtlebot_description/urdf/turtlebot_gazebo.urdf.xacro (robot description, xacro)
@@ -78,19 +78,19 @@
  <gazebo reference="hokuyo_link">
         <sensor type="ray" name="head_hokuyo_sensor">
-          <pose>0 0 0 0 0 0</pose>
+          <pose>0 0 0 0 0 180</pose>
           <visualize>false</visualize>
-          <update_rate>40</update_rate>
+          <update_rate>5.5</update_rate>
           <ray>
             <scan>
               <horizontal>
-                <samples>720</samples>
+                <samples>360</samples>
                 <resolution>1</resolution>
-                <min_angle>-3.1415926</min_angle>
-                <max_angle>3.1415926</max_angle>
+                <min_angle>-3.12414</min_angle>
+                <max_angle>3.14159</max_angle>
               </horizontal>
 </scan>
             <range>
-              <min>0.10</min>
-              <max>30.0</max>
+              <min>0.15</min>
+              <max>12.0</max>
               <resolution>0.01</resolution>
             </range>
@@ -103,5 +103,5 @@
             <plugin name="gazebo_ros_head_hokuyo_controller" filename="libgazebo_ros_laser.so">
             <!--topicName>/turtlebot/laser/scan</topicName-->
-            <topicName>/turtlebot/laser/scan</topicName>
+            <topicName>/scan</topicName>
             <frameName>hokuyo_link</frameName>
         </plugin>
@@ -110,2 +110,38 @@
   </xacro:macro>
 </robot>
+*************************************************************************************************************
+<xacro:macro name="turtlebot_sim_2dsensor">
+ <gazebo reference="laser_link">
+        <sensor type="ray" name="head_rplidar_sensor">
+<!-- 重要理解：定义的雷达其实包括两部分的，一部分是宏sensor_rplidar。另一部分是宏turtlebot_sim_2dsensor，这一部分是不显示的，所以下面visual为false。之间的pose为0 0 0 0 0 0,即两者完全重合-->
+          <pose>0 0 0 0 0 0</pose>
+          <visualize>false</visualize>
+          <update_rate>5.5</update_rate>
+          <ray>
+		    <scan>
+			      <horizontal>
+				<samples>360</samples>
+				<resolution>1</resolution>
+				<min_angle>-3.12414</min_angle>
+				<max_angle>3.14159</max_angle>
+			      </horizontal>
+		    </scan>
+		    <range>
+			      <min>0.15</min>
+			      <max>12.0</max>
+			      <resolution>0.01</resolution>
+		    </range>
+		    <noise>
+			      <type>gaussian</type>
+			       <mean>0.0</mean>
+			      <stddev>0.01</stddev>
+		    </noise>
+          </ray>
+            <plugin name="gazebo_ros_head_hokuyo_controller" filename="libgazebo_ros_laser.so">
+            <!--topicName>/turtlebot/laser/scan</topicName-->
+            <topicName>/scan</topicName>
+            <frameName>laser_link</frameName>
+        </plugin>
+        </sensor>
+      </gazebo>
+  </xacro:macro>

File: turtlebot-kinetic/turtlebot_description/urdf/turtlebot_library.urdf.xacro (robot description, xacro)
@@ -14,8 +14,8 @@
   <xacro:include filename="$(find turtlebot_description)/urdf/stacks/hexagons.urdf.xacro"/>
   <!-- 3D Sensors -->
- <!-- <xacro:include filename="$(find turtlebot_description)/urdf/sensors/kinect.urdf.xacro"/>-->
+ <!-- <xacro:include filename="$(find turtlebot_description)/urdf/sensors/kinect.urdf.xacro"/>
   <xacro:include filename="$(find turtlebot_description)/urdf/sensors/asus_xtion_pro.urdf.xacro"/>
-  <xacro:include filename="$(find turtlebot_description)/urdf/sensors/asus_xtion_pro_offset.urdf.xacro"/>
+  <xacro:include filename="$(find turtlebot_description)/urdf/sensors/asus_xtion_pro_offset.urdf.xacro"/>-->
   <!-- <xacro:include filename="$(find turtlebot_description)/urdf/sensors/rplidar.urdf.xacro"/> -->
-  <xacro:include filename="$(find turtlebot_description)/urdf/sensors/hokuyo.urdf.xacro"/>
+   <!--    <xacro:include filename="$(find turtlebot_description)/urdf/sensors/hokuyo.urdf.xacro"/>-->
 </robot>
